File: hardware/BREAD_Slice.kicad_pcb (KiCad board)
At the start: 2 copper layers, 70 x 100 mm, 22 parts, among them J1 Conn_01x10_Socket, SW1 SW_DIP_x04, U1 AP63205

Commit message: fix(hw): re-point stale library nicknames
These parts exist in KiCad-Master-Lib; the boards referenced libraries that no
longer exist (kml-custom, KML-Custom, and SparkFun libraries that never
contained the part) or names the library has since changed.

KiCad embeds footprint geometry in the .kicad_pcb, so the boards rendered and
fabricated correctly and the rot stayed invisible -- it only surfaces on
update-from-library, or when a generator tries to resolve a nickname.

Nickname/name only. No geometry is changed:

  SparkFun-LED:WS2812-5050-4PIN -> KMLib_IC_SMD:WS2812-5050-4PIN
  kml-custom:AP63205WU-7 -> KMLib_IC_Power:AP63205WU-7_Buck_Regulator
  kml-custom:Arduino_Nano_Headers -> KMLib_Boards_Modules:Arduino_Nano_Headers
  kml-custom:Arduino_Nano_v3.x -> KMLib_IC_MCU_MPU:Arduino_Nano_v3.x
  kml-custom:FAST-Logo-Medium -> KMLib_Aesthetic:FAST-Logo-Medium
  kml-custom:OSHW_Logo_8mm -> KMLib_Aesthetic:OSHW_Logo_8mm
  kml-custom:SOIC_05WU-7_DIO -> KMLib_IC_SMD:SOIC_05WU-7_DIO
  kml-custom:SOIC_05WU-7_DIO-M -> KMLib_IC_SMD:SOIC_05WU-7_DIO-M
  kml-custom:Thermal Pad -> KMLib_Mounting:Thermal_Pad
  kml-custom:WS2812-5050-4PIN -> KMLib_IC_SMD:WS2812-5050-4PIN
  kml-custom:WS2812B_5050 -> SparkFun-LED:WS2812B_5050

Only references that failed to resolve were touched. Generic parts (<=4 pins)
and KiCad *-rescue libraries are deliberately excluded: fingerprint matching
cannot distinguish a 2-pin resistor from a 2-pin capacitor, so those are being
done by hand.
Parts:
- A1: footprint kml-custom:Arduino_Nano_Headers -> KMLib_Boards_Modules:Arduino_Nano_Headers
- D2: footprint kml-custom:WS2812-5050-4PIN -> KMLib_IC_SMD:WS2812-5050-4PIN
- G***: footprint kml-custom:FAST-Logo-Medium -> KMLib_Aesthetic:FAST-Logo-Medium
- HS1: footprint kml-custom:Thermal Pad -> KMLib_Mounting:Thermal_Pad
- Ref**: footprint kml-custom:OSHW_Logo_8mm -> KMLib_Aesthetic:OSHW_Logo_8mm
- U1: footprint kml-custom:SOIC_05WU-7_DIO-M -> KMLib_IC_SMD:SOIC_05WU-7_DIO-M
Changed lines of the file:
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@@
 		)
 	)
-	(footprint "kml-custom:WS2812-5050-4PIN"
+	(footprint "KMLib_IC_SMD:WS2812-5050-4PIN"
 		(locked yes)
 		(layer "F.Cu")
@@
 		)
 	)
-	(footprint "kml-custom:Arduino_Nano_Headers"
+	(footprint "KMLib_Boards_Modules:Arduino_Nano_Headers"
 		(layer "F.Cu")
 		(at 142.61 97.44)
@@
 		)
 	)
-	(footprint "kml-custom:OSHW_Logo_8mm"
+	(footprint "KMLib_Aesthetic:OSHW_Logo_8mm"
 		(layer "F.Cu")
 		(at 135.950001 107.8 -90)
@@
 		(embedded_fonts no)
 	)
-	(footprint "kml-custom:FAST-Logo-Medium"
+	(footprint "KMLib_Aesthetic:FAST-Logo-Medium"
 		(layer "F.Cu")
 		(at 130.1 70.3 -90)
@@
 		(embedded_fonts no)
 	)
-	(footprint "kml-custom:Thermal Pad"
+	(footprint "KMLib_Mounting:Thermal_Pad"
 		(layer "F.Cu")
 		(at 131.8 121.45)
@@
 		)
 	)
-	(footprint "kml-custom:SOIC_05WU-7_DIO-M"
+	(footprint "KMLib_IC_SMD:SOIC_05WU-7_DIO-M"
 		(layer "B.Cu")
 		(at 128.75 122.755)
